File: pathfinder/kicad/papaya-pcb/papaya-pcb.kicad_sch (KiCad schematic)
At the start: 0 parts

Commit message: Add personal README, dev log, and KiCad schematic generator
Split docs into a fork-specific README (this build's hardware/docs/tooling)
and an archived upstream README for attribution. Adds development-log.md
summarizing the wiring model and generator work. Extends
papaya-wiring-layout.yaml with real wire gauges and the UBEC 6V/servo/motor
wiring, and adds generate_schematic.py, which forward-engineers a fully
wired starter KiCad schematic from that YAML (validated against KiCad 10
with zero ERC errors).

Co-Authored-By: Claude Sonnet 5 <noreply@anthropic.com>
Parts:
- added BT1: Main LiPo Battery, symbol AUTO:BT1
- added BTS1: Motor Driver #1 (BTS7960/IBT_2), symbol AUTO:BTS1
- added BTS2: Motor Driver #2 (BTS7960/IBT_2), symbol AUTO:BTS2
- added ELRS1: ELRS Receiver (RadioMaster RP3-V2), symbol AUTO:ELRS1
- added ESP32: ESP32-S3, symbol AUTO:ESP32
- added F1: Main Power Fuse, symbol AUTO:F1
- added J1: J1 (2 pins), symbol AUTO:J1
- added J10: J_S2 (3 pins), symbol AUTO:J10
- added J11: J_S3 (3 pins), symbol AUTO:J11
- added J12: J_S4 (3 pins), symbol AUTO:J12
- added J2: J_ESP32 (13 pins), symbol AUTO:J2
- added J3: J_UBEC5V (4 pins), symbol AUTO:J3
- added J4: J_BTS1 (6 pins), symbol AUTO:J4
- added J5: J_BTS2 (6 pins), symbol AUTO:J5
- added J6: J_ELRS (4 pins), symbol AUTO:J6
- added J7: J_GND_MASTER (1 pins), symbol AUTO:J7
- added J8: J_UBEC6V (2 pins), symbol AUTO:J8
- added J9: J_S1 (3 pins), symbol AUTO:J9
- added M1: Motor 1 (Right - Wheel 1), symbol AUTO:M1
- added M2: Motor 2 (Left - Wheel 2), symbol AUTO:M2
- added M3: Motor 3 (Right - Wheel 3), symbol AUTO:M3
- added M4: Motor 4 (Left - Wheel 4), symbol AUTO:M4
- added M5: Motor 5 (Right - Wheel 5), symbol AUTO:M5
- added M6: Motor 6 (Left - Wheel 6), symbol AUTO:M6
- added S1: Servo 1 (Right-Front - Wheel 1), symbol AUTO:S1
- added S2: Servo 2 (Left-Front - Wheel 2), symbol AUTO:S2
- added S3: Servo 3 (Right-Rear - Wheel 5), symbol AUTO:S3
- added S4: Servo 4 (Left-Rear - Wheel 6), symbol AUTO:S4
- added SW1: Main Power Switch, symbol AUTO:SW1
- added TB1: Power Distribution Terminal Block, symbol AUTO:TB1
- added TB2: Motor Power Distribution Bus, symbol AUTO:TB2
- added U1: UBEC 6V/8A, symbol AUTO:U1
- added U2: UBEC 5V/3A, symbol AUTO:U2
Connections:
- new net NET_A_BUS: BTS1.B+ (Motor supply B+ (screw terminal)), BTS2.B+ (Motor supply B+ (screw terminal)), J1.1 (Main battery power IN (raw 3S voltage, feeds UBEC 5V/3A input)), J3.INP (UBEC 5V IN+ pad), SW1.OUT (Output), TB1.A-IN (A-Master Input), TB1.A12 (A12 - BTS2 supply +), TB1.A13 (A13 - board main power in (feeds UBEC 5V/3A)), TB1.A14, TB1.A6 (A6 - UBEC 6V/8A (U1) input +), TB1.A7 (A7 - BTS1 supply +), U1.IN+ (Input + (red wire)), U2.IN+ (Input +)
- new net NET_BATTERY_MAIN_POS: BT1.POS (Positive (+)), F1.IN (Input (from battery))
- new net NET_BTS1_PIN1_RPWM: BTS1.PIN1_RPWM (Pin 1 - R-PWM), ESP32.GPIO12 (BTS #1 - pin 1), J2.12 (ESP32 GPIO12 - BTS1 pin 1, R-PWM (socket pin)), J4.1 (BTS1 pin 1 - R-PWM)
- new net NET_BTS1_PIN2_LPWM: BTS1.PIN2_LPWM (Pin 2 - L-PWM), ESP32.GPIO13 (BTS #1 - pin 2), J2.13 (ESP32 GPIO13 - BTS1 pin 2, L-PWM (socket pin)), J4.2 (BTS1 pin 2 - L-PWM)
- new net NET_BTS2_PIN1_RPWM: BTS2.PIN1_RPWM (Pin 1 - R-PWM), ESP32.GPIO10 (BTS #2 - pin 1), J2.10 (ESP32 GPIO10 - BTS2 pin 1, R-PWM (socket pin)), J5.1 (BTS2 pin 1 - R-PWM)
- new net NET_BTS2_PIN2_LPWM: BTS2.PIN2_LPWM (Pin 2 - L-PWM), ESP32.GPIO11 (BTS #2 - pin 2), J2.11 (ESP32 GPIO11 - BTS2 pin 2, L-PWM (socket pin)), J5.2 (BTS2 pin 2 - L-PWM)
- new net NET_BUS_5V: BTS1.PIN3_REN (Pin 3 - R-EN), BTS1.PIN4_LEN (Pin 4 - L-EN), BTS1.PIN7_VCC (Pin 7 - VCC), BTS2.PIN3_REN (Pin 3 - R-EN), BTS2.PIN4_LEN (Pin 4 - L-EN), BTS2.PIN7_VCC (Pin 7 - VCC), ELRS1.VCC (VCC (red wire)), ESP32.5V_IN (5V power in), J2.5V (ESP32 5V IN (socket pin)), J3.OUTP (UBEC 5V OUT+ pad), J4.3 (BTS1 pin 3 - R-EN (5V bus)), J4.4 (BTS1 pin 4 - L-EN (5V bus)), J4.7 (BTS1 pin 7 - VCC (5V bus)), J5.3 (BTS2 pin 3 - R-EN (5V bus)), J5.4 (BTS2 pin 4 - L-EN (5V bus)), J5.7 (BTS2 pin 7 - VCC (5V bus)), J6.VCC (ELRS VCC (5V bus)), U2.OUT+ (Output +)
- new net NET_BUS_6V: J10.PWR (S2 header pin 2 - PWR (red)), J11.PWR (S3 header pin 2 - PWR (red)), J12.PWR (S4 header pin 2 - PWR (red)), J8.OUTP (UBEC 6V OUT+ (servo power bus)), J9.PWR (S1 header pin 2 - PWR (red)), S1.PWR (Power (6V)), S2.PWR (Power (6V)), S3.PWR (Power (6V)), S4.PWR (Power (6V)), U1.OUT+ (Output + (6V))
- new net NET_B_BUS: BT1.NEG (Negative (-)), BTS1.B- (Motor supply B- (screw terminal)), BTS1.PIN8_GND (Pin 8 - GND), BTS2.B- (Motor supply B- (screw terminal)), BTS2.PIN8_GND (Pin 8 - GND), ELRS1.GND (GND (black wire)), ESP32.GND_1 (Ground (near 5V IN)), ESP32.GND_2 (Ground (near TX)), J1.2 (J1.2), J10.GND (S2 header pin 1 - GND (black)), J11.GND (S3 header pin 1 - GND (black)), J12.GND (S4 header pin 1 - GND (black)), J2.GND_1 (ESP32 ground, near 5V IN (socket pin)), J2.GND_2 (ESP32 ground, near TX (socket pin)), J3.INN (UBEC 5V IN- pad), J3.OUTN (UBEC 5V OUT- pad), J4.8 (BTS1 pin 8 - GND (ground bus)), J5.8 (BTS2 pin 8 - GND (ground bus)), J6.GND (ELRS GND (ground bus)), J7.1 (Master ground OUT (to tb-power-dist.B14)), J8.OUTN (UBEC 6V OUT- (servo power bus return)), J9.GND (S1 header pin 1 - GND (black)), S1.GND (Ground), S2.GND (Ground), S3.GND (Ground), S4.GND (Ground), TB1.B-IN (B-Master Input), TB1.B12 (B12 - BTS2 supply -), TB1.B13 (B13 - board main power return), TB1.B14 (B14 - board master ground return), TB1.B6 (B6 - UBEC 6V/8A (U1) input -), TB1.B7 (B7 - BTS1 supply -), U1.IN- (Input - (black wire)), U1.OUT- (Output - (6V)), U2.IN- (Input -), U2.OUT- (Output -)
- new net NET_ELRS_RX: ELRS1.RX (RX - receiver input (white wire)), ESP32.GPIO21 (ELRS RX (white wire)), J2.21 (ESP32 GPIO21 - ELRS RX, white wire (socket pin)), J6.RX (ELRS RX (white wire))
- new net NET_ELRS_TX: ELRS1.TX (TX - receiver output (green wire)), ESP32.GPIO47 (ELRS TX (green wire)), J2.47 (ESP32 GPIO47 - ELRS TX, green wire (socket pin)), J6.TX (ELRS TX (green wire))
- new net NET_FUSE_MAIN_OUT: F1.OUT (Output (to switch/distribution)), SW1.IN (Input)
- new net NET_LEFT_POWER: BTS2.M+ (Motor output M+ (screw terminal)), M2.+ (Motor +), M4.+ (Motor +), M6.+ (Motor +), TB2.A5 (Left power - from BTS2 M+ (driver output)), TB2.A6 (Left power - to Motor 2), TB2.A7 (Left power - to Motor 4), TB2.A8 (Left power - to Motor 6)
- new net NET_LEFT_RETURN: BTS2.M- (Motor output M- (screw terminal)), M2.- (Motor -), M4.- (Motor -), M6.- (Motor -), TB2.B5 (Left return - from BTS2 M- (driver output)), TB2.B6 (Left return - from Motor 2), TB2.B7 (Left return - from Motor 4), TB2.B8 (Left return - from Motor 6)
- new net NET_RIGHT_POWER: BTS1.M+ (Motor output M+ (screw terminal)), M1.+ (Motor +), M3.+ (Motor +), M5.+ (Motor +), TB2.A1 (Right power - from BTS1 M+ (driver output)), TB2.A2 (Right power - to Motor 1), TB2.A3 (Right power - to Motor 3), TB2.A4 (Right power - to Motor 5)
- new net NET_RIGHT_RETURN: BTS1.M- (Motor output M- (screw terminal)), M1.- (Motor -), M3.- (Motor -), M5.- (Motor -), TB2.B1 (Right return - from BTS1 M- (driver output)), TB2.B2 (Right return - from Motor 1), TB2.B3 (Right return - from Motor 3), TB2.B4 (Right return - from Motor 5)
- new net NET_S1_SIG: ESP32.GPIO42 (Servo signal - S1 (Right-Front)), J2.42 (ESP32 GPIO42 - S1 (Right-Front) servo signal (socket pin)), J9.SIG (S1 header pin 3 - SIG (white)), S1.SIG (Signal (GPIO42, per ESP32 wiring instructions))
- new net NET_S2_SIG: ESP32.GPIO7 (Servo signal - S2 (Left-Front)), J10.SIG (S2 header pin 3 - SIG (white)), J2.7 (ESP32 GPIO7 (socket pin)), S2.SIG (Signal (GPIO7, per ESP32 wiring instructions))
- new net NET_S3_SIG: ESP32.GPIO41 (Servo signal - S3 (Right-Rear)), J11.SIG (S3 header pin 3 - SIG (white)), J2.41 (ESP32 GPIO41 - S3 (Right-Rear) servo signal (socket pin)), S3.SIG (Signal (GPIO41, per ESP32 wiring instructions))
- new net NET_S4_SIG: ESP32.GPIO38 (Servo signal - S4 (Left-Rear)), J12.SIG (S4 header pin 3 - SIG (white)), J2.38 (ESP32 GPIO38 - S4 (Left-Rear) servo signal (socket pin)), S4.SIG (Signal (GPIO38, per ESP32 wiring instructions))
