File: pathfinder/kicad/papaya-pcb/papaya-pcb.kicad_sch (KiCad schematic)
At the start: 33 parts, among them J1 J1 (2 pins), J10 J_S2 (3 pins), J11 J_S3 (3 pins), J12 J_S4 (3 pins), J2 J_ESP32 (13 pins), J3 J_UBEC5V (4 pins), J4 J_BTS1 (6 pins), J5 J_BTS2 (6 pins), J6 J_ELRS (4 pins), J7 J_GND_MASTER (1 pins), J8 J_UBEC6V (2 pins), J9 J_S1 (3 pins), M1 Motor 1 (Right - Wheel 1), M2 Motor 2 (Left - Wheel 2), M3 Motor 3 (Right - Wheel 3), M4 Motor 4 (Left - Wheel 4), M5 Motor 5 (Right - Wheel 5), M6 Motor 6 (Left - Wheel 6), SW1 Main Power Switch, U1 UBEC 6V/8A, U2 UBEC 5V/3A

Commit message: Update with modified KiCad Schema
Connections:
- net NET_A_BUS: no longer J3.INP (UBEC 5V IN+ pad)
- net NET_B_BUS: no longer J1.2 (J1.2)
- new net: J1.2 (J1.2), J3.INP (U2_5V_IN-POS)
Other:
- moved on the sheet: BT1, BTS1, BTS2, ELRS1, ESP32, F1, J1, J10, J11, J12, J2, J3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
