File: pathfinder/kicad/papaya-pcb/papaya-pcb.kicad_sch (KiCad schematic)
At the start: 33 parts, among them J1 J1 (2 pins), J10 J_S2 (3 pins), J11 J_S3 (3 pins), J12 J_S4 (3 pins), J2 J_ESP32 (13 pins), J3 J_UBEC5V (4 pins), J4 J_BTS1 (6 pins), J5 J_BTS2 (6 pins), J6 J_ELRS (4 pins), J7 J_GND_MASTER (1 pins), J8 J_UBEC6V (2 pins), J9 J_S1 (3 pins), M1 Motor 1 (Right - Wheel 1), M2 Motor 2 (Left - Wheel 2), M3 Motor 3 (Right - Wheel 3), M4 Motor 4 (Left - Wheel 4), M5 Motor 5 (Right - Wheel 5), M6 Motor 6 (Left - Wheel 6), SW1 Main Power Switch, U1 UBEC 6V/8A, U2 UBEC 5V/3A

Commit message: Commit with components on the board pending trace layouts.
Parts:
- J10, J11, J12, J9: footprint Connector_PinHeader_2.54mm:PinHeader_1x03_P2.54mm_Vertical -> papaya-pcb:PinHeader_1x03_Servo
- J4, J5: footprint Connector_PinHeader_2.54mm:PinHeader_1x06_P2.54mm_Vertical -> papaya-pcb:PinHeader_1x06_BTS_Signal
- J6: footprint Connector_PinHeader_2.54mm:PinHeader_1x04_P2.54mm_Vertical -> papaya-pcb:PinHeader_1x04_ELRS
- J8: footprint TerminalBlock:TerminalBlock_MaiXu_MX126-5.0-02P_1x02_P5.00mm -> papaya-pcb:TerminalBlock_2Pos_UBEC6V
Changed lines of the file:
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@@
 			)
 		)
-		(property "Footprint" "Connector_PinHeader_2.54mm:PinHeader_1x03_P2.54mm_Vertical"
+		(property "Footprint" "papaya-pcb:PinHeader_1x03_Servo"
 			(at 309.88 382.27 0)
 			(hide yes)
@@
 			)
 		)
-		(property "Footprint" "Connector_PinHeader_2.54mm:PinHeader_1x03_P2.54mm_Vertical"
+		(property "Footprint" "papaya-pcb:PinHeader_1x03_Servo"
 			(at 224.79 381 0)
 			(hide yes)
@@
 			)
 		)
-		(property "Footprint" "Connector_PinHeader_2.54mm:PinHeader_1x04_P2.54mm_Vertical"
+		(property "Footprint" "papaya-pcb:PinHeader_1x04_ELRS"
 			(at 64.77 260.35 0)
 			(hide yes)
@@
 			)
 		)
-		(property "Footprint" "Connector_PinHeader_2.54mm:PinHeader_1x03_P2.54mm_Vertical"
+		(property "Footprint" "papaya-pcb:PinHeader_1x03_Servo"
 			(at 76.2 379.73 0)
 			(hide yes)
@@
 			)
 		)
-		(property "Footprint" "TerminalBlock:TerminalBlock_MaiXu_MX126-5.0-02P_1x02_P5.00mm"
+		(property "Footprint" "papaya-pcb:TerminalBlock_2Pos_UBEC6V"
 			(at 274.32 166.37 0)
 			(hide yes)
@@
 			)
 		)
-		(property "Footprint" "Connector_PinHeader_2.54mm:PinHeader_1x03_P2.54mm_Vertical"
+		(property "Footprint" "papaya-pcb:PinHeader_1x03_Servo"
 			(at 143.51 381 0)
 			(hide yes)
@@
 			)
 		)
-		(property "Footprint" "Connector_PinHeader_2.54mm:PinHeader_1x06_P2.54mm_Vertical"
+		(property "Footprint" "papaya-pcb:PinHeader_1x06_BTS_Signal"
 			(at 165.1 162.56 0)
 			(hide yes)
@@
 			)
 		)
-		(property "Footprint" "Connector_PinHeader_2.54mm:PinHeader_1x06_P2.54mm_Vertical"
+		(property "Footprint" "papaya-pcb:PinHeader_1x06_BTS_Signal"
 			(at 68.58 158.75 0)
 			(hide yes)
